Commit message: Fix orientation of phone
Use Global Unity frame for translation and local unity for orientation

File: tango_phone.urdf (robot description, URDF)
Before this commit: robot tango_phone, 1 links, 0 joints
Links:
- removed link base_link
- added link phone; visual mesh filename=file:///home/rohan/Tango/tango_phone.dae scale=0.01 0.01 0.01

Commit message: checked in the ologic map, plus rviz template files.

File: tango_phone.urdf (robot description, URDF)
Before this commit: robot tango_phone, 1 links, 0 joints
Links:
- link phone: geometry visual mesh filename=file:///home/brandonb/ROSTango/tango_phone.dae scale=0.01 0.01 0.01
