Commit message: updated the rviz files and urdf link

File: ROSTango/src/tango_bringup/urdf/tango_phone.urdf (robot description, URDF)
Before this commit: robot tango_phone, 1 links, 0 joints
Links:
- link phone: geometry visual mesh filename=package://tango_bringup/urdf/tango_phone.dae scale=0.01 0.01 0.01
